File: bichito_e_luz.kicad_pcb (KiCad board)
At the start: 2 copper layers, 34.5 x 27.2 mm, 14 parts, among them P1 USB_C_Plug, U1 NCP1529

Commit message: Add pulldowns updated values and assembly layer
Signed-off-by: Marcos Chaparro <mchaparro@paltatech.com>
Parts:
- F1: value Polyfuse -> FUSE 1A
- R1: value 330R -> 1R
- R2: value 100k -> 432k
- R3: value 22k -> 100k
Changed lines of the file:
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@@
-(kicad_pcb (version 4) (host pcbnew 4.0.7)
+(kicad_pcb (version 20170920) (host pcbnew no-vcs-found-df472e6~60~ubuntu16.04.1)
   (general
-    (links 27)
-    (no_connects 0)
-    (area 120 86.7 181.000001 150.750001)
     (thickness 0.8)
     (drawings 20)
@@
     (47 F.CrtYd user)
     (48 B.Fab user)
-    (49 F.Fab user hide)
+    (49 F.Fab user)
   )
   (setup
-    (last_trace_width 2)
+    (last_trace_width 0.25)
     (user_trace_width 0.25)
     (user_trace_width 0.5)
@@
     (pad_to_mask_clearance 0.2)
     (aux_axis_origin 0 0)
-    (visible_elements 7FFFFFFF)
+    (visible_elements 7FFFFF7F)
     (pcbplotparams
       (layerselection 0x010f0_80000001)
       (usegerberextensions true)
+      (usegerberattributes true)
+      (usegerberadvancedattributes true)
+      (creategerberjobfile true)
       (excludeedgelayer true)
       (linewidth 0.100000)
@@
       (hpglpenspeed 20)
       (hpglpendiameter 15)
-      (hpglpenoverlay 2)
       (psnegative false)
       (psa4output false)
@@
       (effects (font (size 1 1) (thickness 0.15)))
     )
-    (fp_text value 10uF (at 0 1.75) (layer F.Fab)
-      (effects (font (size 1 1) (thickness 0.15)))
-    )
-    (fp_text user %R (at 0 -1.5) (layer F.Fab)
-      (effects (font (size 1 1) (thickness 0.15)))
+    (fp_text value 10uF (at 0.1 1.4) (layer F.Fab) hide
+      (effects (font (size 1 1) (thickness 0.15)))
+    )
+    (fp_text user %R (at 0 0) (layer F.Fab)
+      (effects (font (size 0.5 0.5) (thickness 0.075)))
     )
     (fp_line (start -1 0.62) (end -1 -0.62) (layer F.Fab) (width 0.1))
@@
       (effects (font (size 1 1) (thickness 0.15)))
     )
-    (fp_text value 1nF (at 0 1.5) (layer F.Fab)
+    (fp_text value 1nF (at 0 -1.1) (layer F.Fab) hide
       (effects (font (size 1 1) (thickness 0.15)))
     )
@@
       (effects (font (size 1 1) (thickness 0.15)))
     )
-    (fp_text value 10uF (at 0 1.75 180) (layer F.Fab)
-      (effects (font (size 1 1) (thickness 0.15)))
-    )
-    (fp_text user %R (at 0 -1.5 180) (layer F.Fab)
-      (effects (font (size 1 1) (thickness 0.15)))
+    (fp_text value 10uF (at 0 1.75 180) (layer F.Fab) hide
+      (effects (font (size 1 1) (thickness 0.15)))
+    )
+    (fp_text user %R (at 0 0 180) (layer F.Fab)
+      (effects (font (size 0.5 0.5) (thickness 0.075)))
     )
     (fp_line (start -1 0.62) (end -1 -0.62) (layer F.Fab) (width 0.1))
@@
       (effects (font (size 1 1) (thickness 0.15)))
     )
-    (fp_text value LED_ALT (at 0 2.25 90) (layer F.Fab)
+    (fp_text value LED_ALT (at 0 2.25 90) (layer F.Fab) hide
       (effects (font (size 1 1) (thickness 0.15)))
     )
@@
       (effects (font (size 1 1) (thickness 0.15)))
     )
-    (fp_text value 10uH (at 0 3.17 90) (layer F.Fab)
+    (fp_text value 10uH (at 0 3.17 90) (layer F.Fab) hide
       (effects (font (size 1 1) (thickness 0.15)))
     )
@@
       (effects (font (size 1 1) (thickness 0.15)))
     )
-    (fp_text value 330R (at 0 2.4 270) (layer F.Fab)
+    (fp_text value 1R (at 0 2.4 270) (layer F.Fab) hide
       (effects (font (size 1 1) (thickness 0.15)))
     )
@@
       (effects (font (size 1 1) (thickness 0.15)))
     )
-    (fp_text value 100k (at 0 1.5) (layer F.Fab)
+    (fp_text value 432k (at -0.4 1.2) (layer F.Fab) hide
       (effects (font (size 1 1) (thickness 0.15)))
     )
@@
       (effects (font (size 1 1) (thickness 0.15)))
     )
-    (fp_text value 22k (at 0 1.5) (layer F.Fab)
+    (fp_text value 100k (at 0.3 1.3) (layer F.Fab) hide
       (effects (font (size 1 1) (thickness 0.15)))
     )
@@
       (effects (font (size 1 1) (thickness 0.15)))
     )
-    (fp_text value NCP1529 (at 0 2.9 180) (layer F.Fab)
+    (fp_text value NCP1529 (at 0 2.9 180) (layer F.Fab) hide
       (effects (font (size 1 1) (thickness 0.15)))
     )
@@
       (effects (font (size 1 1) (thickness 0.15)))
     )
-    (fp_text value USB_C_Plug (at 0 -1.96 90) (layer F.Fab)
-      (effects (font (size 1 1) (thickness 0.15)))
-    )
-    (fp_text user %R (at 0 2.04 90) (layer F.Fab)
+    (fp_text value USB_C_Plug (at 0 -1.96 90) (layer F.Fab) hide
+      (effects (font (size 1 1) (thickness 0.15)))
+    )
+    (fp_text user %R (at 0 0.04 90) (layer F.Fab)
       (effects (font (size 1 1) (thickness 0.1)))
     )
@@
       (effects (font (size 1 1) (thickness 0.15)))
     )
-    (fp_text value Polyfuse (at 0 1.75 180) (layer F.Fab)
-      (effects (font (size 1 1) (thickness 0.15)))
-    )
+    (fp_text value "FUSE 1A" (at 0 1.75 180) (layer F.Fab) hide
+      (effects (font (size 1 1) (thickness 0.15)))
+    )
